File: pcb/termometr.sch (KiCad schematic (older format))
At the start: 100 parts, among them P1 CONN_01X03, P2 CONN_01X03, P3 CONN_01X02, Q1 MMBT2222ALT1G, Q10 MMBT2222ALT1G, Q11 MMBT2222ALT1G, Q12 FDV304P, Q13 FDV304P, Q14 MMBT2222ALT1G, Q15 MMBT2222ALT1G, Q16 MMBT2222ALT1G, Q17 MMBT2222ALT1G, Q2 MMBT2222ALT1G, Q3 MMBT2222ALT1G, Q4 MMBT2222ALT1G, Q5 FDV304P, Q6 MMBT2222ALT1G, Q7 FDV304P, Q8 FDV304P, Q9 FDV304P, U1 LT1009, U10 LM1117, U11 HEF4544B, U2 MCP6031, U3 PT100, U4 MCP6N16, U5 MCP3421A0T-E/CH, U6 STM32M030F4, U7 HEF4544B, U8 3x8, U9 3x8

Commit message: Next version. First iteration.
Parts:
- U8, U9: footprint Displays_7-Segment:Cx56-12 -> footprint:3x7segment
Connections:
- net S2: now also U6.7 (PA1); no longer U6.10 (PA4)
- net S3: now also U6.8 (PA2); no longer U6.9 (PA3)
- net at R22.1: now also U6.10 (PA4); no longer U6.7 (PA1)
- net at R20.1: now also U6.9 (PA3); no longer U6.8 (PA2)
Changed lines of the file:
@@
 F 0 "U8" H 9300 4050 60  0000 C CNN
 F 1 "3x8" H 7800 4050 60  0000 C CNN
-F 2 "Displays_7-Segment:Cx56-12" H 8650 4550 60  0001 C CNN
+F 2 "footprint:3x7segment" H 8650 4550 60  0001 C CNN
 F 3 "" H 8650 4550 60  0000 C CNN
 	1    8500 4650
@@
 F 0 "U9" H 11100 4050 60  0000 C CNN
 F 1 "3x8" H 9600 4050 60  0000 C CNN
-F 2 "Displays_7-Segment:Cx56-12" H 10450 4550 60  0001 C CNN
+F 2 "footprint:3x7segment" H 10450 4550 60  0001 C CNN
 F 3 "" H 10450 4550 60  0000 C CNN
 	1    10300 4650
@@
 	3200 5250 3200 5800
 Wire Wire Line
-	3550 4900 4700 4900
-Wire Wire Line
-	3550 4800 3750 4800
-Wire Wire Line
-	3750 4800 3750 5250
+	3550 4800 5850 4800
 Wire Wire Line
 	3750 5250 3200 5250
 Wire Wire Line
-	3800 4700 3800 5550
-Wire Wire Line
-	3800 5550 4150 5550
+	3600 5550 4150 5550
 Wire Wire Line
 	750  5300 4600 5300
@@
 	4100 5050 4100 5850
 Wire Wire Line
-	3600 5150 3600 5000
-Wire Wire Line
 	3600 5000 3550 5000
 Wire Wire Line
 	1550 4800 1550 7250
 Wire Wire Line
-	3600 5150 1050 5150
+	1050 5150 3800 5150
 Wire Wire Line
 	1050 5150 1050 4700
@@
 Wire Wire Line
 	5200 4200 5900 4200
-Wire Wire Line
-	4700 4900 4700 4800
-Wire Wire Line
-	4700 4800 5850 4800
 Wire Wire Line
 	5900 4200 5900 4700
@@
 	5850 4800 5850 4100
 Connection ~ 5850 4100
+Wire Wire Line
+	3800 5150 3800 4700
+Wire Wire Line
+	3600 5000 3600 5550
+Wire Wire Line
+	3750 5250 3750 4900
+Wire Wire Line
+	3750 4900 3550 4900
 $EndSCHEMATC
